File: MacroBoardPcb.sch (KiCad schematic (older format))
At the start: 32 parts, among them SW1 SW_Push, SW2 Rotary_Encoder_Switch, U1 ATmega32U4-AU, Y1 16MHz

Commit message: finished schematics
Connections:
- net GND: now also SW2.C
- net ROW0: now also SW2.S2, U1.28 (PB4); no longer U1.11 (PB3)
- net ROW1: now also U1.29 (PB5); no longer U1.28 (PB4)
- net S0: now reaches U1.12 (PB7)
- net S0: now also SW2.B
- net S1: now reaches U1.20 (PD2)
- net S1: now also SW2.A
- net COL3: now reaches SW2.S1
- net COL3: now also U1.11 (PB3)
Other:
- note added: "Rotary Encoder w/ Switch\n"
- moved on the sheet: C1, C2, C3, C4, C5, C6, C7, D1, D2, D3, D4, D5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

Commit message: added footprints and fully finished schematics
Parts:
- added C4: 0.1uF, Capacitor_SMD:C_0805_2012Metric, symbol Device:C_Small
- added D7: SOD-123, Diode_SMD:D_SOD-123, symbol Device:D_Small
- added J1: AVR-ISP-6, Connector_PinHeader_2.54mm:PinHeader_2x03_P2.54mm_Vertical, symbol Connector:AVR-ISP-6
- C1, C2, C3: footprint (none) -> Capacitor_SMD:C_0805_2012Metric
- C5: renamed from C4; footprint (none) -> Capacitor_SMD:C_0805_2012Metric
- C6: renamed from C5; footprint (none) -> Capacitor_SMD:C_0805_2012Metric
- C7: renamed from C6; footprint (none) -> Capacitor_SMD:C_0805_2012Metric
- C8: renamed from C7; footprint (none) -> Capacitor_SMD:C_0805_2012Metric
- D1, D2, D3, D4, D5, D6: footprint (none) -> Diode_SMD:D_SOD-123
- MX1, MX2, MX3, MX4, MX5, MX6: footprint (none) -> MX_Alps_Hybrid:MX-1U-NoLED
- OL1: footprint (none) -> kbd:OLED_v2
- R1, R2, R3, R4, R5, R6: footprint (none) -> Resistor_SMD:R_0805_2012Metric
- RV1: footprint (none) -> Potentiometer_THT:Potentiometer_Bourns_PTA6043_Single_Slide
- SW1: footprint (none) -> random-keyboard-parts:SKQG-1155865
- SW2: footprint (none) -> Rotary_Encoder:RotaryEncoder_Alps_EC11E-Switch_Vertical_H20mm
- USB1: footprint (none) -> Type-C:HRO-TYPE-C-31-M-12
- Y1: footprint (none) -> Crystal:Crystal_SMD_3225-4Pin_3.2x2.5mm
Connections:
- net +5V: now also C4.1, J1.2 (VCC)
- net COL0: now also U1.21 (PD3); no longer U1.8 (PB0)
- net COL1: now also U1.25 (PD4); no longer U1.9 (PB1)
- net COL2: now also U1.22 (PD5); no longer U1.10 (PB2)
- net COL3: now also U1.26 (PD6); no longer U1.11 (PB3)
- net GND: now also C4.2, J1.6 (GND)
- net ROW0: now also U1.31 (PC6), D7.1 (K); no longer SW2.S2, U1.28 (PB4)
- net ROW1: now also U1.32 (PC7); no longer U1.29 (PB5)
- net RST: now reaches R6.2, SW1.2, U1.13 (~RESET)
- net RST: now also J1.5 (~RST)
- new net: D7.2 (A), SW2.S2
- new net MISO: J1.1 (MISO), U1.11 (PB3)
- new net MOSI: J1.4 (MOSI), U1.10 (PB2)
- new net SCK: J1.3 (SCK), U1.9 (PB1)
- no-connect marks 0 -> 3
Other:
- note added: "ISP Connector\n"
- moved on the sheet: C1, C2, C3, C5, SW1

Commit message: finished routing
Connections:
- net COL0: now also U1.28 (PB4); no longer U1.21 (PD3)
- net COL1: now also U1.27 (PD7); no longer U1.25 (PD4)
- net COL2: now also U1.26 (PD6); no longer MX3.1 (COL), U1.22 (PD5)
- net COL3: now also MX3.1 (COL), U1.25 (PD4); no longer U1.26 (PD6)
- net ROW0: now also U1.32 (PC7); no longer D3.1 (K), U1.31 (PC6)
- net ROW1: now also D3.1 (K), U1.31 (PC6); no longer U1.32 (PC7)
Changed lines of the file:
@@
 Wire Wire Line
 	6350 4100 6300 4100
-Wire Wire Line
-	7050 3550 6700 3550
 Connection ~ 6300 3550
 Wire Wire Line
 	6300 3550 6200 3550
-Connection ~ 6700 3550
 Wire Wire Line
 	6700 3550 6300 3550
@@
 	1    0    0    -1
 $EndComp
-Wire Wire Line
-	7300 3900 7300 3150
-Connection ~ 7300 3150
-Wire Wire Line
-	7300 3150 7300 2900
 Text GLabel 6550 2900 1    50   Input ~ 0
 COL0
 Text GLabel 6950 2900 1    50   Input ~ 0
 COL1
-Text GLabel 7300 2900 1    50   Input ~ 0
+Text GLabel 7300 3900 1    50   Input ~ 0
 COL2
 Text GLabel 6200 3550 0    50   Input ~ 0
@@
 Wire Notes Line
 	3350 1700 5850 1700
+Text GLabel 5450 3200 2    50   Input ~ 0
+ROW1
 Text GLabel 5450 3300 2    50   Input ~ 0
-ROW1
-Text GLabel 5450 3200 2    50   Input ~ 0
 ROW0
-Text GLabel 5450 4000 2    50   Input ~ 0
+Text GLabel 5450 4100 2    50   Input ~ 0
 COL2
-Text GLabel 5450 3900 2    50   Input ~ 0
+Text GLabel 5450 4200 2    50   Input ~ 0
 COL1
-Text GLabel 5450 3800 2    50   Input ~ 0
+Text GLabel 5450 2700 2    50   Input ~ 0
 COL0
 Text GLabel 6300 5550 2    50   Input ~ 0
@@
 Text Notes 5900 5750 0    50   ~ 0
 Rotary Encoder w/ Switch\n
-Text GLabel 5450 4100 2    50   Input ~ 0
+Text GLabel 5450 3900 2    50   Input ~ 0
 COL3
 Connection ~ 3750 4400
@@
 Text GLabel 8300 5000 0    50   Input ~ 0
 MISO
+Text GLabel 7300 2900 1    50   Input ~ 0
+COL3
+Wire Wire Line
+	7050 3550 7400 3550
+Wire Wire Line
+	7400 3550 7400 4300
+Wire Wire Line
+	7400 4300 7050 4300
+Connection ~ 7050 4300
+Wire Wire Line
+	7300 2900 7300 3150
 $EndSCHEMATC
